Commit message: sim sep

File: robotDog.urdf (robot description, URDF)
Before this commit: robot assembled_robot, 29 links, 28 joints
Links:
- removed link actuator_servo_high_torque_10
- removed link actuator_servo_high_torque_12
- removed link actuator_servo_high_torque_15
- removed link actuator_servo_high_torque_17
- removed link actuator_servo_high_torque_20
- removed link actuator_servo_high_torque_22
- removed link actuator_servo_high_torque_5
- removed link actuator_servo_high_torque_7
- removed link actuator_servo_standard_25
- removed link compute_sbc_small_2
- removed link mobility_rubber_foot_pad_14
- removed link mobility_rubber_foot_pad_19
- removed link mobility_rubber_foot_pad_24
- removed link mobility_rubber_foot_pad_9
- removed link power_lipo_3s_2200_3
- removed link sensor_depth_camera_small_27
- removed link structural_bracket_u_26
- removed link structural_extrusion_2020_11
- removed link structural_extrusion_2020_13
- removed link structural_extrusion_2020_16
- removed link structural_extrusion_2020_18
- removed link structural_extrusion_2020_21
- removed link structural_extrusion_2020_23
- removed link structural_extrusion_2020_6
- removed link structural_extrusion_2020_8
- added link actuator_servo_high_torque_11, mass 0.1650; collision box size=0.046500 0.025840 0.036000; collision box size=0.053475 0.004080 0.036000
- added link actuator_servo_high_torque_16, mass 0.1650; collision box size=0.046500 0.025840 0.036000; collision box size=0.053475 0.004080 0.036000
- added link actuator_servo_high_torque_21, mass 0.1650; collision box size=0.046500 0.025840 0.036000; collision box size=0.053475 0.004080 0.036000
- added link actuator_servo_high_torque_26, mass 0.1650; collision box size=0.046500 0.025840 0.036000; collision box size=0.053475 0.004080 0.036000
- added link actuator_servo_standard_13, mass 0.0550; collision box size=0.040000 0.028120 0.020000; collision box size=0.046000 0.004440 0.020000
- added link actuator_servo_standard_18, mass 0.0550; collision box size=0.040000 0.028120 0.020000; collision box size=0.046000 0.004440 0.020000
- added link actuator_servo_standard_23, mass 0.0550; collision box size=0.040000 0.028120 0.020000; collision box size=0.046000 0.004440 0.020000
- added link actuator_servo_standard_6, mass 0.0550; collision box size=0.040000 0.028120 0.020000; collision box size=0.046000 0.004440 0.020000
- added link actuator_servo_standard_9, mass 0.0550; collision box size=0.040000 0.028120 0.020000; collision box size=0.046000 0.004440 0.020000
- added link compute_sbc_small_3, mass 0.0460; collision box size=0.006800 0.006720 0.005950; collision box size=0.006800 0.006720 0.005950
- added link mobility_rubber_foot_pad_15, mass 0.0200; collision cylinder length=0.002000 radius=0.012000; collision cylinder length=0.005000 radius=0.010000
- added link mobility_rubber_foot_pad_20, mass 0.0200; collision cylinder length=0.002000 radius=0.012000; collision cylinder length=0.005000 radius=0.010000
- added link mobility_rubber_foot_pad_25, mass 0.0200; collision cylinder length=0.002000 radius=0.012000; collision cylinder length=0.005000 radius=0.010000
- added link mobility_rubber_foot_pad_30, mass 0.0200; collision cylinder length=0.002000 radius=0.012000; collision cylinder length=0.005000 radius=0.010000
- added link power_lipo_3s_2200_2, mass 0.1850; collision box size=0.012600 0.002720 0.001440; collision box size=0.021000 0.005100 0.001920
- added link sensor_depth_camera_small_8, mass 0.0720; collision box size=0.013500 0.007500 0.007500; collision box size=0.090000 0.025000 0.025000
- added link sensor_lidar_2d_5, mass 0.1800; collision cylinder length=0.002460 radius=0.038500; collision cylinder length=0.006150 radius=0.036050
- added link structural_bracket_u_7, mass 0.0250; collision box size=0.003000 0.030000 0.040000; collision box size=0.003000 0.030000 0.040000
- added link structural_extrusion_2020_10, mass 0.0540; collision box size=0.004000 0.006000 0.100100; collision box size=0.004000 0.006000 0.100100
- added link structural_extrusion_2020_12, mass 0.0540; collision box size=0.004000 0.006000 0.100100; collision box size=0.004000 0.006000 0.100100
- added link structural_extrusion_2020_14, mass 0.0540; collision box size=0.004000 0.006000 0.080080; collision box size=0.004000 0.006000 0.080080
- added link structural_extrusion_2020_17, mass 0.0540; collision box size=0.004000 0.006000 0.100100; collision box size=0.004000 0.006000 0.100100
- added link structural_extrusion_2020_19, mass 0.0540; collision box size=0.004000 0.006000 0.080080; collision box size=0.004000 0.006000 0.080080
- added link structural_extrusion_2020_22, mass 0.0540; collision box size=0.004000 0.006000 0.100100; collision box size=0.004000 0.006000 0.100100
- added link structural_extrusion_2020_24, mass 0.0540; collision box size=0.004000 0.006000 0.080080; collision box size=0.004000 0.006000 0.080080
- added link structural_extrusion_2020_27, mass 0.0540; collision box size=0.004000 0.006000 0.100100; collision box size=0.004000 0.006000 0.100100
- link structural_extrusion_2020_29: geometry collision box size=0.004000 0.006000 0.080080; collision box size=0.004000 0.006000 0.080080
Joints:
- removed joint joint_actuator_servo_high_torque_10
- removed joint joint_actuator_servo_high_torque_12
- removed joint joint_actuator_servo_high_torque_15
- removed joint joint_actuator_servo_high_torque_17
- removed joint joint_actuator_servo_high_torque_20
- removed joint joint_actuator_servo_high_torque_22
- removed joint joint_actuator_servo_high_torque_5
- removed joint joint_actuator_servo_high_torque_7
- removed joint joint_actuator_servo_standard_25
- removed joint joint_compute_sbc_small_2
- removed joint joint_mobility_rubber_foot_pad_14
- removed joint joint_mobility_rubber_foot_pad_19
- removed joint joint_mobility_rubber_foot_pad_24
- removed joint joint_mobility_rubber_foot_pad_9
- removed joint joint_power_lipo_3s_2200_3
- removed joint joint_sensor_depth_camera_small_27
- removed joint joint_structural_bracket_u_26
- removed joint joint_structural_extrusion_2020_11
- removed joint joint_structural_extrusion_2020_13
- removed joint joint_structural_extrusion_2020_16
- removed joint joint_structural_extrusion_2020_18
- removed joint joint_structural_extrusion_2020_21
- removed joint joint_structural_extrusion_2020_23
- removed joint joint_structural_extrusion_2020_6
- removed joint joint_structural_extrusion_2020_8
- added joint joint_actuator_servo_high_torque_11: type revolute, parent structural_baseplate_1, child actuator_servo_high_torque_11, origin xyz=0.0700 0.0525 -0.0220 rpy=0 0 0, axis 0 1 0, limit lower=-3.14159 upper=3.14159 effort=10.6 velocity=3.14
- added joint joint_actuator_servo_high_torque_16: type revolute, parent structural_baseplate_1, child actuator_servo_high_torque_16, origin xyz=-0.0700 0.0525 -0.0220 rpy=0 0 0, axis 0 1 0, limit lower=-3.14159 upper=3.14159 effort=10.6 velocity=3.14
- added joint joint_actuator_servo_high_torque_21: type revolute, parent structural_baseplate_1, child actuator_servo_high_torque_21, origin xyz=0.0700 -0.0525 -0.0220 rpy=0 0 0, axis 0 1 0, limit lower=-3.14159 upper=3.14159 effort=10.6 velocity=3.14
- added joint joint_actuator_servo_high_torque_26: type revolute, parent structural_baseplate_1, child actuator_servo_high_torque_26, origin xyz=-0.0700 -0.0525 -0.0220 rpy=0 0 0, axis 0 1 0, limit lower=-3.14159 upper=3.14159 effort=10.6 velocity=3.14
- added joint joint_actuator_servo_standard_13: type revolute, parent structural_extrusion_2020_12, child actuator_servo_standard_13, origin xyz=0.0000 0.0000 -0.0685 rpy=0 0 0, axis 0 1 0, limit lower=-3.14159 upper=3.14159 effort=1.5 velocity=3.14
- added joint joint_actuator_servo_standard_18: type revolute, parent structural_extrusion_2020_17, child actuator_servo_standard_18, origin xyz=0.0000 0.0000 -0.0685 rpy=0 0 0, axis 0 1 0, limit lower=-3.14159 upper=3.14159 effort=1.5 velocity=3.14
- added joint joint_actuator_servo_standard_23: type revolute, parent structural_extrusion_2020_22, child actuator_servo_standard_23, origin xyz=0.0000 0.0000 -0.0685 rpy=0 0 0, axis 0 1 0, limit lower=-3.14159 upper=3.14159 effort=1.5 velocity=3.14
- added joint joint_actuator_servo_standard_6: type revolute, parent structural_baseplate_1, child actuator_servo_standard_6, origin xyz=0.1200 0.0000 0.0000 rpy=0 0 0, axis 0 1 0, limit lower=-3.14159 upper=3.14159 effort=1.5 velocity=3.14
- added joint joint_actuator_servo_standard_9: type revolute, parent structural_baseplate_1, child actuator_servo_standard_9, origin xyz=-0.1200 0.0000 0.0000 rpy=0 0 0, axis 0 0 1, limit lower=-3.14159 upper=3.14159 effort=1.5 velocity=3.14
- added joint joint_compute_sbc_small_3: type fixed, parent structural_baseplate_1, child compute_sbc_small_3, origin xyz=-0.0700 0.0525 0.0135 rpy=0 0 0, axis 0 0 1
- added joint joint_mobility_rubber_foot_pad_15: type fixed, parent structural_extrusion_2020_14, child mobility_rubber_foot_pad_15, origin xyz=0.0000 0.0000 -0.0475 rpy=0 0 0, axis 0 0 1
- added joint joint_mobility_rubber_foot_pad_20: type fixed, parent structural_extrusion_2020_19, child mobility_rubber_foot_pad_20, origin xyz=0.0000 0.0000 -0.0475 rpy=0 0 0, axis 0 0 1
- added joint joint_mobility_rubber_foot_pad_25: type fixed, parent structural_extrusion_2020_24, child mobility_rubber_foot_pad_25, origin xyz=0.0000 0.0000 -0.0475 rpy=0 0 0, axis 0 0 1
- added joint joint_mobility_rubber_foot_pad_30: type fixed, parent structural_extrusion_2020_29, child mobility_rubber_foot_pad_30, origin xyz=0.0000 0.0000 -0.0475 rpy=0 0 0, axis 0 0 1
- added joint joint_power_lipo_3s_2200_2: type fixed, parent structural_baseplate_1, child power_lipo_3s_2200_2, origin xyz=0.0700 0.0525 0.0170 rpy=0 0 0, axis 0 0 1
- added joint joint_sensor_depth_camera_small_8: type fixed, parent structural_bracket_u_7, child sensor_depth_camera_small_8, origin xyz=0.0700 0.0000 -0.0035 rpy=0 0.1745 0, axis 0 0 1
- added joint joint_sensor_lidar_2d_5: type fixed, parent structural_baseplate_1, child sensor_lidar_2d_5, origin xyz=-0.0700 -0.0525 0.0255 rpy=0 0 0, axis 0 0 1
- added joint joint_structural_bracket_u_7: type fixed, parent actuator_servo_standard_6, child structural_bracket_u_7, origin xyz=0.0000 0.0000 0.0300 rpy=0 0 0, axis 0 0 1
- added joint joint_structural_extrusion_2020_10: type fixed, parent actuator_servo_standard_9, child structural_extrusion_2020_10, origin xyz=-0.0330 0.0000 0.0000 rpy=0 0 0, axis 0 0 1
- added joint joint_structural_extrusion_2020_12: type fixed, parent actuator_servo_high_torque_11, child structural_extrusion_2020_12, origin xyz=0.0000 0.0000 -0.0680 rpy=0 0 0, axis 0 0 1
- added joint joint_structural_extrusion_2020_14: type fixed, parent actuator_servo_standard_13, child structural_extrusion_2020_14, origin xyz=0.0000 0.0000 -0.0500 rpy=0 0 0, axis 0 0 1
- added joint joint_structural_extrusion_2020_17: type fixed, parent actuator_servo_high_torque_16, child structural_extrusion_2020_17, origin xyz=0.0000 0.0000 -0.0680 rpy=0 0 0, axis 0 0 1
- added joint joint_structural_extrusion_2020_19: type fixed, parent actuator_servo_standard_18, child structural_extrusion_2020_19, origin xyz=0.0000 0.0000 -0.0500 rpy=0 0 0, axis 0 0 1
- added joint joint_structural_extrusion_2020_22: type fixed, parent actuator_servo_high_torque_21, child structural_extrusion_2020_22, origin xyz=0.0000 0.0000 -0.0680 rpy=0 0 0, axis 0 0 1
- added joint joint_structural_extrusion_2020_24: type fixed, parent actuator_servo_standard_23, child structural_extrusion_2020_24, origin xyz=0.0000 0.0000 -0.0500 rpy=0 0 0, axis 0 0 1
- added joint joint_structural_extrusion_2020_27: type fixed, parent actuator_servo_high_torque_26, child structural_extrusion_2020_27, origin xyz=0.0000 0.0000 -0.0680 rpy=0 0 0, axis 0 0 1
- joint joint_actuator_servo_standard_28: axis 0 0 1 -> 0 1 0; origin xyz=-0.1200 0.0000 0.0000 rpy=0 0 0 -> xyz=0.0000 0.0000 -0.0685 rpy=0 0 0; parent structural_baseplate_1 -> structural_extrusion_2020_27
- joint joint_sensor_imu_6dof_4: origin xyz=0.0700 -0.0262 0.0065 rpy=0 0 0 -> xyz=0.0700 -0.0525 0.0065 rpy=0 0 0
- joint joint_structural_extrusion_2020_29: origin xyz=-0.0330 0.0000 0.0000 rpy=0 0 0 -> xyz=0.0000 0.0000 -0.0500 rpy=0 0 0
