Commit message: temp

File: car.urdf (robot description, URDF)
Before this commit: robot assembled_robot, 13 links, 12 joints
Links:
- removed link compute_motor_driver_dual_8
- removed link compute_sbc_small_7
- removed link mobility_wheel_driven_2
- removed link mobility_wheel_driven_3
- removed link mobility_wheel_driven_5
- removed link power_distribution_unit_13
- removed link power_lipo_4s_5000_6
- removed link sensor_depth_camera_small_11
- removed link sensor_imu_6dof_9
- removed link sensor_lidar_2d_10
- removed link sensor_ultrasonic_12
- removed link structural_baseplate_1
- added link compute_motor_driver_dual_26, mass 0.0280; collision box size=0.010750 0.006450 0.007500; collision box size=0.017200 0.017200 0.006000
- added link compute_sbc_small_27, mass 0.0460; collision box size=0.006800 0.006720 0.005950; collision box size=0.006800 0.006720 0.005950
- added link mobility_wheel_driven_10, mass 0.1200; collision cylinder length=0.030000 radius=0.050000; collision cylinder length=0.031500 radius=0.017500
- added link mobility_wheel_driven_13, mass 0.1200; collision cylinder length=0.030000 radius=0.050000; collision cylinder length=0.031500 radius=0.017500
- added link mobility_wheel_driven_16, mass 0.1200; collision cylinder length=0.030000 radius=0.050000; collision cylinder length=0.031500 radius=0.017500
- added link mobility_wheel_driven_19, mass 0.1200; collision cylinder length=0.030000 radius=0.050000; collision cylinder length=0.031500 radius=0.017500
- added link mobility_wheel_driven_7, mass 0.1200; collision cylinder length=0.030000 radius=0.050000; collision cylinder length=0.031500 radius=0.017500
- added link motor_gear_medium_37mm_12, mass 0.1800; collision box size=0.025900 0.025900 0.028000; collision cylinder length=0.014000 radius=0.002590
- added link motor_gear_medium_37mm_15, mass 0.1800; collision box size=0.025900 0.025900 0.028000; collision cylinder length=0.014000 radius=0.002590
- added link motor_gear_medium_37mm_18, mass 0.1800; collision box size=0.025900 0.025900 0.028000; collision cylinder length=0.014000 radius=0.002590
- added link motor_gear_medium_37mm_3, mass 0.1800; collision box size=0.025900 0.025900 0.028000; collision cylinder length=0.014000 radius=0.002590
- added link motor_gear_medium_37mm_6, mass 0.1800; collision box size=0.025900 0.025900 0.028000; collision cylinder length=0.014000 radius=0.002590
- added link motor_gear_medium_37mm_9, mass 0.1800; collision box size=0.025900 0.025900 0.028000; collision cylinder length=0.014000 radius=0.002590
- added link power_distribution_unit_25, mass 0.0600; collision box size=0.065000 0.045000 0.015000; visual box size=0.065000 0.045000 0.015000
- added link power_lipo_4s_5000_24, mass 0.4200; collision box size=0.016440 0.003360 0.001800; collision box size=0.027400 0.006300 0.002400
- added link sensor_depth_camera_small_21, mass 0.0720; collision box size=0.013500 0.007500 0.007500; collision box size=0.090000 0.025000 0.025000
- added link sensor_imu_6dof_23, mass 0.0030; collision box size=0.004000 0.002400 0.001500; collision box size=0.006400 0.006400 0.001200
- added link sensor_lidar_2d_20, mass 0.1800; collision cylinder length=0.002460 radius=0.038500; collision cylinder length=0.006150 radius=0.036050
- added link sensor_ultrasonic_22, mass 0.0080; collision box size=0.045000 0.020000 0.015000; collision cylinder length=0.002250 radius=0.004400
- added link structural_baseplate_large_1, mass 2.1000; collision box size=0.350000 0.250000 0.008000; collision cylinder length=0.008080 radius=0.010000
- added link structural_servo_coupler_disc_11, mass 0.0150; collision cylinder length=0.008000 radius=0.016000; visual cylinder length=0.008000 radius=0.016000
- added link structural_servo_coupler_disc_14, mass 0.0150; collision cylinder length=0.008000 radius=0.016000; visual cylinder length=0.008000 radius=0.016000
- added link structural_servo_coupler_disc_17, mass 0.0150; collision cylinder length=0.008000 radius=0.016000; visual cylinder length=0.008000 radius=0.016000
- added link structural_servo_coupler_disc_2, mass 0.0150; collision cylinder length=0.008000 radius=0.016000; visual cylinder length=0.008000 radius=0.016000
- added link structural_servo_coupler_disc_5, mass 0.0150; collision cylinder length=0.008000 radius=0.016000; visual cylinder length=0.008000 radius=0.016000
- added link structural_servo_coupler_disc_8, mass 0.0150; collision cylinder length=0.008000 radius=0.016000; visual cylinder length=0.008000 radius=0.016000
Joints:
- removed joint joint_compute_motor_driver_dual_8
- removed joint joint_compute_sbc_small_7
- removed joint joint_mobility_wheel_driven_2
- removed joint joint_mobility_wheel_driven_3
- removed joint joint_mobility_wheel_driven_5
- removed joint joint_power_distribution_unit_13
- removed joint joint_power_lipo_4s_5000_6
- removed joint joint_sensor_depth_camera_small_11
- removed joint joint_sensor_imu_6dof_9
- removed joint joint_sensor_lidar_2d_10
- removed joint joint_sensor_ultrasonic_12
- added joint joint_compute_motor_driver_dual_26: type fixed, parent structural_baseplate_large_1, child compute_motor_driver_dual_26, origin xyz=0.0000 -0.0875 0.0115 rpy=0 0 0, axis 0 0 1
- added joint joint_compute_sbc_small_27: type fixed, parent structural_baseplate_large_1, child compute_sbc_small_27, origin xyz=0.1225 -0.0875 0.0066 rpy=0 0 0, axis 0 0 1
- added joint joint_mobility_wheel_driven_10: type fixed, parent motor_gear_medium_37mm_9, child mobility_wheel_driven_10, origin xyz=0.0000 0.0000 -0.0990 rpy=-1.5708 0.0000 0.0000, axis 0 1 0
- added joint joint_mobility_wheel_driven_13: type fixed, parent motor_gear_medium_37mm_12, child mobility_wheel_driven_13, origin xyz=0.0000 0.0000 -0.0990 rpy=-1.5708 0.0000 0.0000, axis 0 1 0
- added joint joint_mobility_wheel_driven_16: type fixed, parent motor_gear_medium_37mm_15, child mobility_wheel_driven_16, origin xyz=0.0000 0.0000 -0.0990 rpy=-1.5708 0.0000 0.0000, axis 0 1 0
- added joint joint_mobility_wheel_driven_19: type fixed, parent motor_gear_medium_37mm_18, child mobility_wheel_driven_19, origin xyz=0.0000 0.0000 -0.0990 rpy=-1.5708 0.0000 0.0000, axis 0 1 0
- added joint joint_mobility_wheel_driven_7: type fixed, parent motor_gear_medium_37mm_6, child mobility_wheel_driven_7, origin xyz=0.0000 0.0000 -0.0990 rpy=-1.5708 0.0000 0.0000, axis 0 1 0
- added joint joint_motor_gear_medium_37mm_12: type revolute, parent structural_servo_coupler_disc_11, child motor_gear_medium_37mm_12, origin xyz=0.0000 0.0000 -0.0530 rpy=0.0000 0.0000 0.0000, axis 0 1 0, limit lower=-3.14159 upper=3.14159 effort=10 velocity=3.14
- added joint joint_motor_gear_medium_37mm_15: type revolute, parent structural_servo_coupler_disc_14, child motor_gear_medium_37mm_15, origin xyz=0.0000 0.0000 -0.0530 rpy=0.0000 0.0000 0.0000, axis 0 1 0, limit lower=-3.14159 upper=3.14159 effort=10 velocity=3.14
- added joint joint_motor_gear_medium_37mm_18: type revolute, parent structural_servo_coupler_disc_17, child motor_gear_medium_37mm_18, origin xyz=0.0000 0.0000 -0.0530 rpy=0.0000 0.0000 0.0000, axis 0 1 0, limit lower=-3.14159 upper=3.14159 effort=10 velocity=3.14
- added joint joint_motor_gear_medium_37mm_3: type revolute, parent structural_servo_coupler_disc_2, child motor_gear_medium_37mm_3, origin xyz=0.0000 0.0000 -0.0530 rpy=0.0000 0.0000 0.0000, axis 0 1 0, limit lower=-3.14159 upper=3.14159 effort=10 velocity=3.14
- added joint joint_motor_gear_medium_37mm_6: type revolute, parent structural_servo_coupler_disc_5, child motor_gear_medium_37mm_6, origin xyz=0.0000 0.0000 -0.0530 rpy=0.0000 0.0000 0.0000, axis 0 1 0, limit lower=-3.14159 upper=3.14159 effort=10 velocity=3.14
- added joint joint_motor_gear_medium_37mm_9: type revolute, parent structural_servo_coupler_disc_8, child motor_gear_medium_37mm_9, origin xyz=0.0000 0.0000 -0.0530 rpy=0.0000 0.0000 0.0000, axis 0 1 0, limit lower=-3.14159 upper=3.14159 effort=10 velocity=3.14
- added joint joint_power_distribution_unit_25: type fixed, parent structural_baseplate_large_1, child power_distribution_unit_25, origin xyz=-0.1225 -0.0875 0.0115 rpy=0 0 0, axis 0 0 1
- added joint joint_power_lipo_4s_5000_24: type fixed, parent structural_baseplate_large_1, child power_lipo_4s_5000_24, origin xyz=0.1225 0.0875 0.0190 rpy=0 0 0, axis 0 0 1
- added joint joint_sensor_depth_camera_small_21: type fixed, parent structural_baseplate_large_1, child sensor_depth_camera_small_21, origin xyz=0.2200 0.0000 -0.0453 rpy=0 0.2618 0, axis 0 0 1
- added joint joint_sensor_imu_6dof_23: type fixed, parent structural_baseplate_large_1, child sensor_imu_6dof_23, origin xyz=0.0000 0.0875 0.0055 rpy=0 0 0, axis 0 0 1
- added joint joint_sensor_lidar_2d_20: type fixed, parent structural_baseplate_large_1, child sensor_lidar_2d_20, origin xyz=-0.1225 0.0875 0.0209 rpy=0 0 0, axis 0 0 1
- added joint joint_sensor_ultrasonic_22: type fixed, parent structural_baseplate_large_1, child sensor_ultrasonic_22, origin xyz=-0.1975 0.0000 0.0000 rpy=0 0 0, axis 0 0 1
- added joint joint_structural_servo_coupler_disc_11: type fixed, parent structural_baseplate_large_1, child structural_servo_coupler_disc_11, origin xyz=-0.1225 -0.0875 -0.0080 rpy=0.0000 0.0000 0.0000, axis 0 0 1
- added joint joint_structural_servo_coupler_disc_14: type fixed, parent structural_baseplate_large_1, child structural_servo_coupler_disc_14, origin xyz=0.0000 -0.0875 -0.0080 rpy=0.0000 0.0000 0.0000, axis 0 0 1
- added joint joint_structural_servo_coupler_disc_17: type fixed, parent structural_baseplate_large_1, child structural_servo_coupler_disc_17, origin xyz=0.1225 -0.0875 -0.0080 rpy=0.0000 0.0000 0.0000, axis 0 0 1
- added joint joint_structural_servo_coupler_disc_2: type fixed, parent structural_baseplate_large_1, child structural_servo_coupler_disc_2, origin xyz=-0.1225 0.0875 -0.0080 rpy=0.0000 0.0000 0.0000, axis 0 0 1
- added joint joint_structural_servo_coupler_disc_5: type fixed, parent structural_baseplate_large_1, child structural_servo_coupler_disc_5, origin xyz=0.0000 0.0875 -0.0080 rpy=0.0000 0.0000 0.0000, axis 0 0 1
- added joint joint_structural_servo_coupler_disc_8: type fixed, parent structural_baseplate_large_1, child structural_servo_coupler_disc_8, origin xyz=0.1225 0.0875 -0.0080 rpy=0.0000 0.0000 0.0000, axis 0 0 1
- joint joint_mobility_wheel_driven_4: limit lower=-3.14159 upper=3.14159 effort=10 velocity=3.14 -> (none); origin xyz=0.1225 -0.0875 -0.0540 rpy=-1.5708 0.0000 0.0000 -> xyz=0.0000 0.0000 -0.0990 rpy=-1.5708 0.0000 0.0000; parent structural_baseplate_1 -> motor_gear_medium_37mm_3; type revolute -> fixed
